Commit message: Added lidar to turtlebot

File: src/basic_mobile_robot/urdf/basic_mobile_robot.urdf (robot description, URDF)
Before this commit: robot basic_mobile_robot, 4 links, 3 joints
Links:
- added link lidar_link, mass 0.1; visual cylinder length=0.05 radius=0.04
Joints:
- added joint lidar_joint: type fixed, parent base_link, child lidar_link, origin xyz=0 0 0.12 rpy=0 0 0
- joint caster_joint: type fix -> fixed
